Commit message: fourth commit

File: mycobot_description/urdf/320_urdf/mycobot_pro_320.urdf (robot description, URDF)
Before this commit: robot firefighter, 9 links, 8 joints
Links:
- removed link world
- added link link10; collision cylinder length=0.0225 radius=0.026; visual cylinder length=0.02 radius=0.026
- added link link7; collision cylinder length=0.015 radius=0.024; visual cylinder length=0.01 radius=0.02
- added link link8; collision box size=0.07 0.04 0.01; visual box size=0.1 0.04 0.01
- added link link9; collision cylinder length=0.02 radius=0.09
- link base: mass 1 -> None; geometry collision cylinder length=0.102 radius=0.0725; visual mesh filename=package://mycobot_description/urdf/320_urdf/base.dae
- link gripper: mass 0.1 -> None; geometry collision mesh filename=package://mycobot_description/urdf/320_urdf/gripper.dae; visual mesh filename=package://mycobot_description/urdf/320_urdf/gripper.dae
- link link1: mass 0.5 -> None; geometry collision cylinder length=0.106 radius=0.043; visual mesh filename=package://mycobot_description/urdf/320_urdf/link1.dae
- link link2: mass 0.4 -> None; geometry collision cylinder length=0.18 radius=0.036; visual mesh filename=package://mycobot_description/urdf/320_urdf/link2.dae
- link link3: mass 0.4 -> None; geometry collision cylinder length=0.14 radius=0.0305; visual mesh filename=package://mycobot_description/urdf/320_urdf/link3.dae
- link link4: mass 0.3 -> None; geometry collision cylinder length=0.083 radius=0.029; visual mesh filename=package://mycobot_description/urdf/320_urdf/link4.dae
- link link5: mass 0.1 -> None; geometry collision cylinder length=0.0849 radius=0.029; visual mesh filename=package://mycobot_description/urdf/320_urdf/link5.dae
- link link6: mass 0.1 -> None
Joints:
- removed joint vitual_joint
- added joint gitpper_to_joint7camera: type fixed, parent gripper, child link7, origin xyz=0 0 0 rpy=0 0 3.14 , axis 0 0 0, limit lower=-3.14 upper=3.14159 effort=1000.0 velocity=0
- added joint gitpper_to_joint8camera: type fixed, parent link7, child link8, origin xyz=0 0 0 rpy=0 0 0 , axis 0 0 0, limit lower=-3.14 upper=3.14159 effort=1000.0 velocity=0
- added joint gitpper_to_joint9: type fixed, parent gripper, child link9, origin xyz=0 0.04 0.03 rpy=0 0 0 , axis 0 0 0, limit lower=-3.14 upper=3.14159 effort=1000.0 velocity=0
- added joint joint6output_to_joint10: type revolute, parent link5, child link10, origin xyz=0 -0.041 0 rpy=-1.57080 0 0 , axis 0 0 1, limit lower=-3 upper=3 effort=1000.0 velocity=0.2
- joint gitpper_to_joint6output: limit (none) -> lower=-3.14 upper=3.14159 effort=1000.0 velocity=0
- joint joint2_to_joint1: limit lower=-3.14 upper=3.14159 effort=1000.0 velocity=0 -> lower=-2.92 upper=2.92 effort=1000.0 velocity=0.2
- joint joint3_to_joint2: limit lower=-3.14 upper=3.14159 effort=1000.0 velocity=0 -> lower=-2.75 upper=2.75 effort=1000.0 velocity=0.2
- joint joint4_to_joint3: limit lower=-3.14 upper=3.14159 effort=1000.0 velocity=0 -> lower=-2.75 upper=2.75 effort=1000.0 velocity=0.2
- joint joint5_to_joint4: limit lower=-3.14 upper=3.14159 effort=1000.0 velocity=0 -> lower=-2.75 upper=2.75 effort=1000.0 velocity=0.2
- joint joint6_to_joint5: limit lower=-3.14 upper=3.14159 effort=1000.0 velocity=0 -> lower=-2.92 upper=2.92 effort=1000.0 velocity=0.2
- joint joint6output_to_joint6: limit lower=-3.14 upper=3.14159 effort=1000.0 velocity=0 -> lower=-3 upper=3 effort=1000.0 velocity=0.2; origin xyz=0 0.06 0 rpy=-1.57080 3.14 0  -> xyz=0 0.06 0 rpy=-1.57080 0 0 

File: mycobot_description/urdf/320_urdf/mycobot_pro_320_gripper.urdf (robot description, URDF)
Before this commit: robot firefighter, 12 links, 11 joints
Joints:
- joint joint2_to_joint1: limit lower=-3.14 upper=3.14159 effort=1000.0 velocity=0 -> lower=-2.92 upper=2.92 effort=1000.0 velocity=0
- joint joint3_to_joint2: limit lower=-3.14 upper=3.14159 effort=1000.0 velocity=0 -> lower=-2.75 upper=2.75 effort=1000.0 velocity=0
- joint joint4_to_joint3: limit lower=-3.14 upper=3.14159 effort=1000.0 velocity=0 -> lower=-2.75 upper=2.75 effort=1000.0 velocity=0
- joint joint5_to_joint4: limit lower=-3.14 upper=3.14159 effort=1000.0 velocity=0 -> lower=-2.75 upper=2.75 effort=1000.0 velocity=0
- joint joint6_to_joint5: limit lower=-3.14 upper=3.14159 effort=1000.0 velocity=0 -> lower=-2.92 upper=2.92 effort=1000.0 velocity=0
- joint joint6output_to_joint6: limit lower=-3.14 upper=3.14159 effort=1000.0 velocity=0 -> lower=-3 upper=3 effort=1000.0 velocity=0

File: mycobot_description/urdf/320_urdf/mycobot_pro_320_legrip_2robo_belt.urdf (robot description, URDF)
Before this commit: robot firefighter, 31 links, 30 joints
Links:
- link base: geometry collision cylinder length=0.102 radius=0.0725; visual mesh filename=package://mycobot_description/urdf/320_urdf/Base_edited_EBP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
- link base2: geometry collision cylinder length=0.102 radius=0.0725; visual mesh filename=package://mycobot_description/urdf/320_urdf/Base_edited_EBP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
- link link1: geometry collision cylinder length=0.106 radius=0.043; visual mesh filename=package://mycobot_description/urdf/320_urdf/link1_edited_EB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
- link link12: geometry collision cylinder length=0.106 radius=0.043; visual mesh filename=package://mycobot_description/urdf/320_urdf/link1_edited_EB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
- link link2: geometry collision cylinder length=0.18 radius=0.036; visual mesh filename=package://mycobot_description/urdf/320_urdf/link2_edited_EB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
- link link22: geometry collision cylinder length=0.18 radius=0.036; visual mesh filename=package://mycobot_description/urdf/320_urdf/link2_edited_EB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
- link link3: geometry collision cylinder length=0.14 radius=0.0305; visual mesh filename=package://mycobot_description/urdf/320_urdf/link3_edited_EB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
- link link32: geometry collision cylinder length=0.14 radius=0.0305; visual mesh filename=package://mycobot_description/urdf/320_urdf/link3_edited_EB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
- link link4: geometry collision cylinder length=0.083 radius=0.029; visual mesh filename=package://mycobot_description/urdf/320_urdf/link4_edited_EB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
- link link42: geometry collision cylinder length=0.083 radius=0.029; visual mesh filename=package://mycobot_description/urdf/320_urdf/link4_edited_EB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
- link link5: geometry collision cylinder length=0.0849 radius=0.029; visual cylinder length=0.002 radius=0.026
- link link52: geometry collision cylinder length=0.0849 radius=0.029; visual cylinder length=0.002 radius=0.026
Joints:
- joint joint2_to_joint1: limit lower=-3.14 upper=3.14159 effort=1000.0 velocity=1.0 -> lower=-2.92 upper=2.92 effort=1000.0 velocity=1.0
- joint joint3_to_joint2: limit lower=-3.14 upper=3.14159 effort=1000.0 velocity=0.4 -> lower=-2.75 upper=2.75 effort=1000.0 velocity=0.6
- joint joint4_to_joint3: limit lower=-3.14 upper=3.14159 effort=1000.0 velocity=0.4 -> lower=-2.75 upper=2.75 effort=1000.0 velocity=0.6
- joint joint5_to_joint4: limit lower=-3.14 upper=3.14159 effort=1000.0 velocity=1.0 -> lower=-2.75 upper=2.75 effort=1000.0 velocity=1.0
- joint joint6_to_joint5: limit lower=-3.14 upper=3.14159 effort=1000.0 velocity=1.0 -> lower=-2.92 upper=2.92 effort=1000.0 velocity=1.0
- joint joint6output_to_joint6: axis 0 0 1 -> 0 0 -1; limit lower=-3.14 upper=3.14159 effort=1000.0 velocity=1.0 -> lower=-3 upper=3 effort=1000.0 velocity=1.0

File: mycobot_description/urdf/320_urdf/mycobot_pro_320_legrip_writing.urdf (robot description, URDF)
Before this commit: robot firefighter, 16 links, 15 joints
Links:
- removed link pen1
- removed link pen2
- added link link8; collision box size=0.07 0.04 0.01; visual box size=0.1 0.04 0.01
- added link link9; collision cylinder length=0.015 radius=0.024; visual cylinder length=0.01 radius=0.02
- link base: geometry collision cylinder length=0.102 radius=0.0725; visual mesh filename=package://mycobot_description/urdf/320_urdf/Base_edited_EBP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
- link gripper: geometry collision mesh filename=package://mycobot_description/urdf/320_urdf/gripper_leial.d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 scale=1.15 1.15 1.15; visual mesh filename=package://mycobot_description/urdf/320_urdf/gripper_leial.d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 scale=1.15 1.15 1.15
- link leftfinger: geometry collision mesh filename=package://mycobot_description/urdf/320_urdf/dedo_gripper_le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 scale=1.15 1.15 1.15; visual mesh filename=package://mycobot_description/urdf/320_urdf/dedo_gripper_le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 scale=1.15 1.15 1.15
- link link1: geometry collision cylinder length=0.106 radius=0.043; visual mesh filename=package://mycobot_description/urdf/320_urdf/link1_edited_EB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
- link link2: geometry collision cylinder length=0.18 radius=0.036; visual mesh filename=package://mycobot_description/urdf/320_urdf/link2_edited_EB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
- link link3: geometry collision cylinder length=0.14 radius=0.0305; visual mesh filename=package://mycobot_description/urdf/320_urdf/link3_edited_EB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
- link link4: geometry collision cylinder length=0.083 radius=0.029; visual mesh filename=package://mycobot_description/urdf/320_urdf/link4_edited_EB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
- link link5: geometry collision cylinder length=0.0849 radius=0.029; visual cylinder length=0.002 radius=0.026
- link rightfinger: geometry collision mesh filename=package://mycobot_description/urdf/320_urdf/dedo_gripper_le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 scale=1.15 1.15 1.15; visual mesh filename=package://mycobot_description/urdf/320_urdf/dedo_gripper_le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 scale=1.15 1.15 1.15
Joints:
- removed joint gripper_to_pen1
- removed joint gripper_to_pen2
- added joint gitpper_to_joint8camera: type fixed, parent link9, child link8, origin xyz=0 0 0 rpy=0 0 0 , axis 0 0 0, limit lower=-3.14 upper=3.14159 effort=1000.0 velocity=0
- added joint gitpper_to_joint9camera: type fixed, parent gripper, child link9, origin xyz=0 0 0 rpy=0 0 3.14 , axis 0 0 0, limit lower=-3.14 upper=3.14159 effort=1000.0 velocity=0
- joint finger_joint1: origin xyz=0 0 0 rpy=0 0 0 -> xyz=0 -0.01 0 rpy=0 0 0
- joint finger_joint2: origin xyz=0 0 0 rpy=0 0 0 -> xyz=0 -0.01 0 rpy=0 0 0
- joint gripper_to_joint6output: origin xyz=0 0 0 rpy=0 0 3.14  -> xyz=0 0 0 rpy=0 0 0 
- joint joint2_to_joint1: limit lower=-3.14 upper=3.14159 effort=1000.0 velocity=1.0 -> lower=-2.92 upper=2.92 effort=1000.0 velocity=0.5
- joint joint3_to_joint2: limit lower=-3.14 upper=3.14159 effort=1000.0 velocity=0.4 -> lower=-2.75 upper=2.75 effort=1000.0 velocity=0.5
- joint joint4_to_joint3: limit lower=-3.14 upper=3.14159 effort=1000.0 velocity=0.4 -> lower=-2.75 upper=2.75 effort=1000.0 velocity=0.5
- joint joint5_to_joint4: limit lower=-3.14 upper=3.14159 effort=1000.0 velocity=1.0 -> lower=-2.75 upper=2.75 effort=1000.0 velocity=1.0
- joint joint6_to_joint5: limit lower=-3.14 upper=3.14159 effort=1000.0 velocity=1.0 -> lower=-2.92 upper=2.92 effort=1000.0 velocity=1.0; origin xyz=0 -0.0847 0 rpy=1.57080 -1.57080 0 -> xyz=0 -0.0847 0 rpy=1.57080 1.57080 0
- joint joint6output_to_joint6: limit lower=-3.14 upper=3.14159 effort=1000.0 velocity=1.0 -> lower=-3 upper=3 effort=1000.0 velocity=1.0

File: xarm_description/urdf/lite6_robot.urdf.xacro (robot description, xacro)
@@ -16,8 +16,8 @@
   <xacro:arg name="geometry_width" default="0.1"/>
   <xacro:arg name="geometry_mesh_filename" default=""/>
-  <xacro:arg name="geometry_mesh_origin_xyz" default="'0 0 0'"/>
-  <xacro:arg name="geometry_mesh_origin_rpy" default="'0 0 0'"/>
-  <xacro:arg name="geometry_mesh_tcp_xyz" default="'0 0 0'"/>
-  <xacro:arg name="geometry_mesh_tcp_rpy" default="'0 0 0'"/>
+  <xacro:arg name="geometry_mesh_origin_xyz" default="0 0 0"/>
+  <xacro:arg name="geometry_mesh_origin_rpy" default="0 0 0"/>
+  <xacro:arg name="geometry_mesh_tcp_xyz" default="0 0 0"/>
+  <xacro:arg name="geometry_mesh_tcp_rpy" default="0 0 0"/>
   <xacro:arg name="add_realsense_d435i" default="false"/>
   <!-- Añadimos objeto en el escenario -->

File: xarm_description/urdf/lite6_robot_mig.urdf.xacro (robot description, xacro)
@@ -65,5 +65,5 @@
     objeto_length="$(arg objeto_length)" objeto_width="$(arg objeto_width)" />
   <xacro:if value="$(arg add_gripper)">
-    <xacro:include filename="$(find xarm_description)/urdf/lite_gripper.urdf.xacro" />
+    <xacro:include filename="$(find xarm_description)/urdf/lite_gripper_mig.urdf.xacro" />
     <xacro:uflite_gripper_urdf attach_to="$(arg prefix)link_eef" />
   </xacro:if>
